File: PID temperature controller.sch (EAGLE design)
At the start: 12 parts, among them IC1 MAX6675

Commit message: Eagle Schematic and Brd file added
Eagle Schematic and Brd file added
Parts:
- removed SG1: EB2209A, buzzer:EB2209A
- removed THERMOCUPPLE: (no value), con-amp-mt:S02P
- added POWERIN: 5 V, con-amp:MTA02-100
- added R10: 0 Ohm, adafruit:R-US_0207/12
- added R4: 100 Ohm, resistor-power:RRS1/8
- added R5: 0 Ohm, resistor-power:RRS1/8
- added R7, R8, R9: 10k, resistor-power:RRS1/8
- added SG2: B/C11S, buzzer:B/C11S
- added X1: (no value), con-ptr500:AK300/2
- IC1: device max6675:MAX6675 -> MAX6675:MAX6675
- R2, R3: value 100k -> 100 Ohm
- renumbered MT1 to ENCODER
Connections:
- removed net N$12: ENCODER.B, U$1.IO4
- new net N$17: R4.2, SG2.1
- new net N$18: R10.1, R7.2, R8.2, R9.2
- new net N$20: ENCODER.B, R9.1, U$1.IO2
- new net N$21: ENCODER.A, R8.1, U$1.IO4
- net GND: now also POWERIN.2, SG2.2, U$1.GND@1, U$1.GND@2; no longer SG1.-, U$1.GND
- net N$10: now also R5.1, R7.1; no longer U$1.IO15
- net N$11: now also R5.2, U$1.IO15; no longer ENCODER.A, U$1.IO2
- net N$4: now also R4.1; no longer SG1.+
- net N$5: now also X1-2.KL; no longer THERMOCUPPLE-2.S
- net N$6: now also X1-1.KL; no longer THERMOCUPPLE-1.S
- net N$9: now also U$1.IO32; no longer U$1.IO18
- net VCC: now also POWERIN.1, R10.2
Other:
- note added: "PID-temperature-controller-using-esp32 Ver 2023-04 https://github.com/almorawaka/ESP32"
